File: kicad/backplane/backplane.kicad_sch (KiCad schematic)
At the start: 56 parts, among them J1 Board Connector, J2 Board Connector, J3 Board Connector, J4 Board Connector, J5 Board Connector, J6 Board Connector, J7 Board Connector, J8 Conn_02x04_Counter_Clockwise, J9 Screw_Terminal_01x02, SW1 SW_SPDT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

Commit message: integrated wozmon, updated kicad to specify phi1o
Parts:
- removed C9: 0.1u, Capacitor_THT:C_Disc_D3.8mm_W2.6mm_P2.50mm, symbol Device:C
- removed J8: Conn_02x04_Counter_Clockwise, Connector_IDC:IDC-Header_2x04_P2.54mm_Vertical, symbol Connector_Generic:Conn_02x04_Counter_Clockwise
- removed U1: 7414, Package_DIP:DIP-14_W7.62mm_Socket, symbol 74xx_IEEE:7414
Connections:
- net PHI2 renamed PHI1
- no-connect marks 5 -> 1
