File: kicad/cpu/cpu.kicad_pcb (KiCad board)
At the start: 2 copper layers, 102.5 x 30 mm, 10 parts, among them J1 Board Connector, J8 Conn_02x04_Counter_Clockwise, U1 W65C02SxP

Commit message: integrated wozmon, updated kicad to specify phi1o
Connections:
- net PHI2 renamed PHI1
Changed lines of the file:
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@@
 			(layers "*.Cu" "*.Mask")
 			(remove_unused_layers no)
-			(net "PHI2")
+			(net "PHI1")
 			(pinfunction "ϕ1_3")
 			(pintype "output")
@@
 			(layers "*.Cu" "*.Mask")
 			(remove_unused_layers no)
-			(net "PHI2")
+			(net "PHI1")
 			(pinfunction "Pin_23_23")
 			(pintype "passive")
@@
 	)
 	(segment
-		(start 129.5 107.25)
-		(end 131 108.75)
+		(start 114.315635 105.75)
+		(end 82.75 105.75)
 		(width 0.2)
 		(layer "F.Cu")
-		(net "PHI2")
+		(net "PHI_IN")
 	)
 	(segment
-		(start 129.39 126.49)
-		(end 127.63 128.25)
+		(start 126.96 122.49)
+		(end 115.36 110.89)
 		(width 0.2)
 		(layer "F.Cu")
-		(net "PHI2")
+		(net "PHI_IN")
 	)
 	(segment
-		(start 131 113.818828)
-		(end 139.15 121.968829)
+		(start 115.36 110.89)
+		(end 115.36 106.794365)
 		(width 0.2)
 		(layer "F.Cu")
-		(net "PHI2")
+		(net "PHI_IN")
 	)
 	(segment
-		(start 139.15 123.576855)
-		(end 136.236854 126.49)
-		(width 0.2)
+		(start 72.165 118.205)
+		(end 72.165 118.865)
+		(width 0.5)
 		(layer "F.Cu")
-		(net "PHI2")
+		(net "PHI_IN")
 	)
 	(segment
-		(start 139.15 121.968829)
-		(end 139.15 123.576855)
+		(start 115.36 106.794365)
+		(end 114.315635 105.75)
 		(width 0.2)
 		(layer "F.Cu")
-		(net "PHI2")
+		(net "PHI_IN")
+	)
+	(via
+		(at 82.75 105.75)
+		(size 0.6)
+		(drill 0.3)
+		(layers "F.Cu" "B.Cu")
+		(net "PHI_IN")
 	)
 	(segment
-		(start 136.236854 126.49)
-		(end 129.39 126.49)
+		(start 82.75 115)
+		(end 76.25 121.5)
 		(width 0.2)
-		(layer "F.Cu")
-		(net "PHI2")
+		(layer "B.Cu")
+		(net "PHI_IN")
 	)
 	(segment
-		(start 131 108.75)
-		(end 131 113.818828)
+		(start 74.257919 121.5)
+		(end 72.165 119.407081)
 		(width 0.2)
-		(layer "F.Cu")
-		(net "PHI2")
+		(layer "B.Cu")
+		(net "PHI_IN")
+	)
+	(segment
+		(start 72.165 119.407081)
+		(end 72.165 118.205)
+		(width 0.2)
+		(layer "B.Cu")
+		(net "PHI_IN")
+	)
+	(segment
+		(start 76.25 121.5)
+		(end 74.257919 121.5)
+		(width 0.2)
+		(layer "B.Cu")
+		(net "PHI_IN")
+	)
+	(segment
+		(start 82.75 105.75)
+		(end 82.75 115)
+		(width 0.2)
+		(layer "B.Cu")
+		(net "PHI_IN")
 	)
 	(segment
@@
 	)
 	(segment
-		(start 114.315635 105.75)
-		(end 82.75 105.75)
+		(start 129.5 107.25)
+		(end 131 108.75)
 		(width 0.2)
 		(layer "F.Cu")
-		(net "PHI_IN")
+		(net "PHI1")
 	)
 	(segment
-		(start 126.96 122.49)
-		(end 115.36 110.89)
+		(start 129.39 126.49)
+		(end 127.63 128.25)
 		(width 0.2)
 		(layer "F.Cu")
-		(net "PHI_IN")
+		(net "PHI1")
 	)
 	(segment
-		(start 115.36 110.89)
-		(end 115.36 106.794365)
+		(start 131 113.818828)
+		(end 139.15 121.968829)
 		(width 0.2)
 		(layer "F.Cu")
-		(net "PHI_IN")
+		(net "PHI1")
 	)
 	(segment
-		(start 72.165 118.205)
-		(end 72.165 118.865)
-		(width 0.5)
-		(layer "F.Cu")
-		(net "PHI_IN")
-	)
-	(segment
-		(start 115.36 106.794365)
-		(end 114.315635 105.75)
+		(start 139.15 123.576855)
+		(end 136.236854 126.49)
 		(width 0.2)
 		(layer "F.Cu")
-		(net "PHI_IN")
-	)
-	(via
-		(at 82.75 105.75)
-		(size 0.6)
-		(drill 0.3)
-		(layers "F.Cu" "B.Cu")
-		(net "PHI_IN")
+		(net "PHI1")
 	)
 	(segment
-		(start 82.75 115)
-		(end 76.25 121.5)
-		(width 0.2)
-		(layer "B.Cu")
-		(net "PHI_IN")
-	)
-	(segment
-		(start 74.257919 121.5)
-		(end 72.165 119.407081)
-		(width 0.2)
-		(layer "B.Cu")
-		(net "PHI_IN")
-	)
-	(segment
-		(start 72.165 119.407081)
-		(end 72.165 118.205)
+		(start 139.15 121.968829)
+		(end 139.15 123.576855)
 		(width 0.2)
-		(layer "B.Cu")
-		(net "PHI_IN")
+		(layer "F.Cu")
+		(net "PHI1")
 	)
 	(segment
-		(start 76.25 121.5)
-		(end 74.257919 121.5)
+		(start 136.236854 126.49)
+		(end 129.39 126.49)
 		(width 0.2)
-		(layer "B.Cu")
-		(net "PHI_IN")
+		(layer "F.Cu")
+		(net "PHI1")
 	)
 	(segment
-		(start 82.75 105.75)
-		(end 82.75 115)
+		(start 131 108.75)
+		(end 131 113.818828)
 		(width 0.2)
-		(layer "B.Cu")
-		(net "PHI_IN")
+		(layer "F.Cu")
+		(net "PHI1")
 	)
 	(zone
