File: kicad/mmu/mmu.kicad_pcb (KiCad board)
At the start: 2 copper layers, 102.5 x 30 mm, 22 parts, among them J1 Board Connector, U1 74LS682, U2 74LS139

Commit message: integrated wozmon, updated kicad to specify phi1o
Connections:
- net PHI2 renamed PHI1
Changed lines of the file:
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@@
 			(layers "*.Cu" "*.Mask")
 			(remove_unused_layers no)
-			(net "PHI2")
+			(net "PHI1")
 			(pinfunction "E_15")
 			(pintype "input")
@@
 			(layers "*.Cu" "*.Mask")
 			(remove_unused_layers no)
-			(net "PHI2")
+			(net "PHI1")
 			(pinfunction "Pin_23_23")
 			(pintype "passive")
@@
 	)
 	(segment
+		(start 158.2875 119.107143)
+		(end 160.425 119.107143)
+		(width 0.25)
+		(layer "F.Cu")
+		(net "Net-(D2-A)")
+	)
+	(segment
 		(start 129.875 126.005)
 		(end 127.63 128.25)
 		(width 0.25)
 		(layer "F.Cu")
-		(net "PHI2")
+		(net "PHI1")
 	)
 	(segment
@@
 		(width 0.25)
 		(layer "F.Cu")
-		(net "PHI2")
+		(net "PHI1")
 	)
 	(segment
@@
 		(width 0.25)
 		(layer "F.Cu")
-		(net "PHI2")
-	)
-	(segment
-		(start 158.2875 119.107143)
-		(end 160.425 119.107143)
-		(width 0.25)
-		(layer "F.Cu")
-		(net "Net-(D2-A)")
+		(net "PHI1")
 	)
 	(zone
