File: kicad/mmu/mmu.kicad_sch (KiCad schematic)
At the start: 22 parts, among them J1 Board Connector, U1 74LS682, U2 74LS139

Commit message: integrated wozmon, updated kicad to specify phi1o
Connections:
- net PHI2 renamed PHI1
Changed lines of the file:
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@@
 		)
 	)
-	(global_label "PHI2"
+	(global_label "PHI1"
 		(shape input)
 		(at 180.34 87.63 180)
@@
 		)
 	)
-	(global_label "PHI2"
+	(global_label "PHI1"
 		(shape input)
 		(at 242.57 101.6 180)
