File: kicad/ram/ram.kicad_pcb (KiCad board)
At the start: 2 copper layers, 102.5 x 30 mm, 5 parts, among them J1 Board Connector, U1 7400, U2 AS6C4008-55PCN

Commit message: integrated wozmon, updated kicad to specify phi1o
Connections:
- net PHI2 renamed PHI1
Changed lines of the file:
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@@
 			(layers "*.Cu" "*.Mask")
 			(remove_unused_layers no)
-			(net "PHI2")
+			(net "PHI1")
 			(pinfunction "Pin_23_23")
 			(pintype "passive")
