File: kicad/ram/ram.kicad_sch (KiCad schematic)
At the start: 5 parts, among them J1 Board Connector, U1 7400, U2 AS6C4008-55PCN

Commit message: integrated wozmon, updated kicad to specify phi1o
Connections:
- net PHI2 renamed PHI1
Changed lines of the file:
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@@
 		)
 	)
-	(global_label "PHI2"
+	(global_label "PHI1"
 		(shape input)
 		(at 242.57 101.6 180)
