File: kicad/template/template.kicad_pcb (KiCad board)
At the start: 2 copper layers, 102.5 x 30 mm, 1 part, among them J1 Board Connector

Commit message: added acia board
Connections:
- net PHI2 renamed PHI1
Changed lines of the file:
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@@
 			(layers "*.Cu" "*.Mask")
 			(remove_unused_layers no)
-			(net "PHI2")
+			(net "PHI1")
 			(pinfunction "Pin_23_23")
 			(pintype "passive")
