File: kicad/de9/de9.kicad_pcb (KiCad board)
At the start: 2 copper layers, 49.5 x 30 mm, 7 parts, among them J1 SPI 1, J2 Terminal, J3 SPI 2

Commit message: added spi and via boards
Parts:
- J1, J3: footprint Connector_JST:JST_PH_B6B-PH-K_1x06_P2.00mm_Vertical -> Connector_JST:JST_XH_B6B-XH-AM_1x06_P2.50mm_Vertical
- moved J1 5.51 mm to (117.7, 105.5)
- moved J3 4.26 mm to (139.0, 105.5)
Routing:
- net MISO: track 34.7 -> 29.9 mm
- net MOSI: track 34.7 -> 30.3 mm
- net SCK: track 34.7 -> 30.3 mm
- net EVE_CSB: track 16.9 -> 12.7 mm
- net KBD_CSB: track 22.1 -> 18.3 mm
- net GND: vias 12 -> 15
